File: PCB/TRX/KiCAD/TRX_klopik.sch (KiCad schematic (older format))
At the start: 166 parts, among them J1 MIC, J10 Conn_01x01, J11 Conn_01x01, J12 BPF, J13 AF, J2 OUT, J3 13.6v, J4 RF, J5 Conn_01x05, J6 TX, J7 S-metr, J8 Conn_01x01, J9 Conn_01x01, K1 TQ2-12VDC, Q1 MMBT2222LT1G, Q10 BC847, Q11 BC847, Q12 BC847, Q2 BC857, Q3 BC857, Q4 BC857, Q5 BC847, Q6 BC847, Q7 BC847, Q8 2N7002, Q9 2N7002, T1 Transformer_1P_2S, T2 Transformer_1P_2S, T3 1_4, U1 ADE-1H+, U3 LM386, Y1 8.867Mhz, Y10 8.867Mhz, Y11 8.867Mhz, Y12 8.867Mhz, Y13 8.867Mhz, Y14 8.867Mhz, Y15 8.867Mhz, Y16 8.867Mhz, Y17 8.867Mhz, Y18 8.867Mhz, Y19 8.867Mhz, Y2 8.867Mhz, Y20 8.867Mhz, Y21 8.867Mhz, Y3 8.867Mhz, Y4 8.867Mhz, Y5 8.867Mhz, Y6 8.867Mhz, Y7 8.867Mhz, Y8 8.867Mhz, Y9 8.867Mhz

Commit message: add TRX PCB v1.15
Parts:
- removed C21: 56, TRX_klopik:C_1206_0603, symbol C_Small
- removed C28: 62, TRX_klopik:C_1206_0603, symbol C_Small
- removed D2, D5, D7: LL4148, Diodes_SMD:D_MiniMELF_Handsoldering, symbol D_Small
- removed J12: BPF, Pin_Headers:Pin_Header_Straight_2x06_Pitch2.54mm, symbol Conn_02x06_Odd_Even
- removed J13: AF, Pin_Headers:Pin_Header_Straight_1x03_Pitch2.54mm, symbol Conn_01x03
- removed J4: RF, Pin_Headers:Pin_Header_Angled_1x03_Pitch2.54mm, symbol Conn_01x03
- removed J5: Conn_01x05, Pin_Headers:Pin_Header_Straight_1x05_Pitch2.54mm, symbol Conn_01x05
- removed Q2: BC857, TO_SOT_Packages_SMD:SOT-23_Handsoldering, symbol BFT92
- removed U1: ADE-1H+, TRX_klopik:CD636, symbol ADE-1H+
- removed Y1, Y2, Y3, Y4: 8.867Mhz, TRX_klopik:Crystal_HC49-U_Vertical, symbol Crystal_Filter
- added C48: 47uF, Capacitors_ThroughHole:CP_Radial_D6.3mm_P2.50mm, symbol CP_Small
- added C49: 10uF, Capacitors_Tantalum_SMD:CP_Tantalum_Case-A_EIA-3216-18_Hand, symbol CP_Small
- added D18, D20: D_Small, Diodes_ThroughHole:D_DO-35_SOD27_P7.62mm_Horizontal, symbol D_Small
- added D19: LL4148, Diodes_SMD:D_MiniMELF_Handsoldering, symbol D_Small
- added D2, D5, D7: BAV99, TO_SOT_Packages_SMD:SOT-23_Handsoldering, symbol D_Schottky_x2_Serial_AKC
- added J12: VFO, TRX_klopik:RFCONNECTOR, symbol Conn_01x02
- added J13: VOX, Pin_Headers:Pin_Header_Straight_1x02_Pitch2.54mm, symbol Conn_01x02
- added J14: BFO, Pin_Headers:Pin_Header_Straight_1x02_Pitch2.54mm, symbol Conn_01x02
- added J15: AGC, Pin_Headers:Pin_Header_Straight_1x02_Pitch2.54mm, symbol Conn_01x02
- added J4: BPF, TRX_klopik:RFCONNECTOR, symbol Conn_01x02
- added J5: AUDIO IN, Pin_Headers:Pin_Header_Straight_1x02_Pitch2.54mm, symbol Conn_01x02
- added Q13, Q14: BC847, TO_SOT_Packages_SMD:SOT-23_Handsoldering, symbol BFR92
- added Q2: BC857, TO_SOT_Packages_SMD:SOT-23_Handsoldering, symbol BC857
- added R46: 1k, TRX_klopik:R_1206_0603, symbol R_Small
- added R47, R48, R49: 0R, TRX_klopik:R_1206_0603, symbol R_Small
- added RV3: 200R, Potentiometers:Potentiometer_Trimmer_Piher_PT-6v_Horizontal, symbol POT_TRIM
- added RV4: POT_Dual, TRX_klopik:Potentiometer_WH148_Double, symbol POT_Dual
- added T4, T5: Transformer_1P_2S, TRX_klopik:HF_transf3, symbol Transformer_1P_2S
- C18, C37: value 100nF -> 10nF; footprint TRX_klopik:C_1206_0603 -> Capacitors_SMD:C_0603_HandSoldering
- C20, C34, C57: footprint Capacitors_Tantalum_SMD:CP_Tantalum_Case-D_EIA-7343-31_Hand -> Capacitors_ThroughHole:CP_Radial_D6.3mm_P2.50mm
- C22: value 62 -> 100nF
- C39: value 10uF -> 22uF
- C47: value 100nF -> 330nF
- C6: value 56 -> 100nF
- C8: value 15nF -> 10nF; footprint TRX_klopik:C_1206_0603 -> Capacitors_SMD:C_0603_HandSoldering
- D14, D4: value LL4148 -> D_Small; footprint Diodes_SMD:D_MiniMELF_Handsoldering -> Diodes_ThroughHole:D_DO-35_SOD27_P7.62mm_Horizontal
- D15, D16, D17, D9: value LL4148 -> 1N4148; footprint Diodes_SMD:D_MiniMELF_Handsoldering -> Diodes_ThroughHole:D_DO-35_SOD27_P7.62mm_Horizontal
- Q1: value MMBT2222LT1G -> BC847
- R15: value 680 -> 1k
- R32: value 10 -> 100k
- R33: value 100R -> 300k
- R34: value 20k -> 6.2k
- R35, RV2: value 100 -> 1k
- R39: value 150k -> 2.4k
- R40: value 8k2 -> 330k
- R41: value 15k -> 330R
- R42: value 1k -> 4.7k
- R43: value 470R -> 680R
- R44: value 0 -> 0R
- T1, T2: footprint TRX_klopik:HF12 -> TRX_klopik:HF_transf3
- T3: footprint TRX_klopik:1_4 -> TRX_klopik:TF14
Connections:
- net BFO is gone; now on an unnamed net: R44.1
- net 13.6V: now also C6.1, R39.1, D19.1 (K); no longer C18.1, D15.1 (K), R40.1
- net GND: now also C18.1, C6.2, Q10.2 (E), RV2.1, RV2.2, C48.2, D7.1 (A), J12.2 (Pin_2), J13.2 (Pin_2), J14.2 (Pin_2), J15.2 (Pin_2), J4.2 (Pin_2), J5.2 (Pin_2), Q13.2 (E), Q14.2 (E), RV3.2, RV3.3, RV4.1, RV4.4, T4.2 (AB), T5.2 (AB), T5.4 (SB), T5.5 (SC); no longer C18.2, C6.1, R15.2, R32.2, R35.2, R41.2, R42.2, RV2.3
- net RELAY: now also D19.2 (A); no longer D15.2 (A)
- net TX: now also R41.2; no longer R33.2
- net at C15.1, Q5.1 (B), R18.1: now also Q2.3 (C)
- net at C15.2: now also T4.4 (SB), T4.5 (SC)
- net at R18.2, R19.2: now also D5.1 (A)
- net at C14.1, Q5.3 (C), R11.2: now also Q2.1 (B)
- net at R11.1, R19.1: now also D2.2 (K)
- net at R4.2, R5.2: now also Q2.2 (E)
- net at D1.1 (K): now also D2.1 (A)
- net at C23.2, Y6.2, Y7.1: now also Y5.2
- net at C27.2, Y10.2, Y11.1: now also Y12.1
- net at Y11.2: now also C53.2, Y12.2; no longer Y12.1
- net at D9.2 (A): now also D15.1 (K), T5.3 (SA)
- net at D11.2 (A): now also D5.2 (K); no longer D9.1 (K)
- net at C4.1: now also T4.1 (AA)
- net at C4.2: now also J4.1 (Pin_1)
- net at C29.2, Y14.2, Y15.1: now also Y13.2
- net at Y14.1: now also C17.2, Y13.1; no longer Y13.2
- net at C32.2, Y21.2: now also Y20.2
- net at C35.2, R23.2: now also R49.1
- net at C39.2: now also RV3.1; no longer R35.1
- net at C34.2: now also RV4.3, RV4.6
- net at C42.1, D13.2 (K), Q8.1 (G)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: now also R30.1; no longer R39.1
- net at J2.2 (R), J2.3 (RN), J2.4 (SN)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: now also RV4.2, RV4.5
- net at Q10.1 (B): now also R32.2, R40.1; no longer R39.2
- net at Q10.3 (C), R40.2: now also R39.2, C49.1
- net at C47.2, J1.2 (R), J1.3 (RN)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: now also R42.2
- net at C14.2, Y5.1: now also Y6.1
- net at R8.1: now also J6.1 (Pin_1); no longer Q1.1 (B)
- net at C8.2, R8.2: now also R15.1; no longer R30.1
- net at Q12.1 (B), R34.2: now also R33.1, Q13.3 (C); no longer C47.1, R41.1
- net at C46.1, Q12.3 (C), R34.1: now also C22.2, R41.1, R42.1; no longer R33.1
- net at C5.2, Y19.2, Y20.1: now also Y21.1
- net at C31.1, T2.1 (AA): now also J14.1 (Pin_1); no longer R44.2
- net at D14.1 (K), T2.3 (SA): now also D20.2 (A); no longer D17.2 (A)
- net at D4.2 (A), T2.6 (SD): now also D18.1 (K); no longer D16.1 (K)
- net at C19.1, C31.2, C33.2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: now also RV2.3; no longer R15.1
- net at C7.1: now also T5.1 (AA)
- net at J7.1 (Pin_1): now also C48.1, D7.2 (K); no longer RV2.2
- net at R30.2: now also Q14.3 (C); no longer J6.1 (Pin_1)
- net VFO: no longer names the net of C7.2
- net VFO: now also J12.1 (Pin_1)
- new net: C47.1, Q13.1 (B), R33.2
- new net: D18.2 (A), D20.1 (K), T1.3 (SA)
- new net: D16.2 (A), D9.1 (K), T4.3 (SA)
- new net: D15.2 (A), D17.1 (K), T4.6 (SD)
- new net: D16.1 (K), D17.2 (A), T5.6 (SD)
- new net: C49.2, D7.3 (common)
- new net: Q1.1 (B), R15.2
- new net: J13.1 (Pin_1), R47.2
- new net: J5.1 (Pin_1), R48.2
- new net: Q14.1 (B), R46.1
- new net: C18.2, R35.1, R46.2
- new net: J15.1 (Pin_1), R35.2
- new net: R44.2, R47.1
- new net: R48.1, R49.2
Other:
- note added: "QER filter 8867kHz -3db 2.7kHz Z=260R\n"
- note removed: "QER filter 8Mhz -6db 3 kHz Z=200R\n"
- moved on the sheet: C1, C10, C11, C12, C13, C14, C15, C16, C17, C19, C2, C20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
